File: cubesat_board/cubesat_board.sch (KiCad schematic (older format))
At the start: 2 parts, among them J1 CONN_02X26, J2 CONN_02X26

Commit message: Forgot to previously saver files, slight update
Parts:
- J1, J2: footprint (none) -> Pin_Headers:Pin_Header_Straight_2x26_Pitch2.54mm
Changed lines of the file:
@@
 F 0 "J1" H 8000 4550 50  0000 C CNN
 F 1 "CONN_02X26" V 8000 3200 50  0000 C CNN
-F 2 "" H 8000 2500 50  0001 C CNN
+F 2 "Pin_Headers:Pin_Header_Straight_2x26_Pitch2.54mm" H 8000 2500 50  0001 C CNN
 F 3 "" H 8000 2500 50  0001 C CNN
 	1    8000 3200
@@
 F 0 "J2" H 9850 4550 50  0000 C CNN
 F 1 "CONN_02X26" V 9850 3200 50  0000 C CNN
-F 2 "" H 9850 2500 50  0001 C CNN
+F 2 "Pin_Headers:Pin_Header_Straight_2x26_Pitch2.54mm" H 9850 2500 50  0001 C CNN
 F 3 "" H 9850 2500 50  0001 C CNN
 	1    9850 3200
