File: cubesat_board/cubesat_board.sch (KiCad schematic (older format))
At the start: 2 parts, among them J1 CONN_02X26, J2 CONN_02X26

Commit message: Started defining cubesat bus nets
Parts:
- removed J1, J2: CONN_02X26, Pin_Headers:Pin_Header_Straight_2x26_Pitch2.54mm, symbol CONN_02X26
- added J? (x2): Conn_02x26_Odd_Even, symbol conn:Conn_02x26_Odd_Even
Connections:
- net labels added: +3V3, +5V, 1-WIRE, ADC_INT, BAT_HTR_EN_1, BAT_HTR_EN_2, BAT_HTR_EN_3, BAT_HTR_EN_4, BAT_HTR_MUX_SEL, BAT_HTR_STAT_1, BAT_HTR_STAT_2, BAT_HTR_STAT_3, BAT_HTR_STAT_4, DEPLOYMENT_A, DEPLOYMENT_B, GND, He_EN, He_Tx_I_SENSE, He_UART_RX, He_UART_TX, PAYLOAD_ACT, PAYLOAD_EN, PAYLOAD_HTR, PAYLOAD_I_SENSE, SC4, SCL, SCL_B, SD4, SDA, SDA_B, SOLAR_BACK_NEG, SOLAR_BACK_POS, SOLAR_FRONT_NEG, SOLAR_FRONT_POS, SOLAR_LEFT_NEG, SOLAR_LEFT_POS, SOLAR_RIGHT_NEG, SOLAR_RIGHT_POS, VAA
- wire segments 0 -> 63

Commit message: Changed some nets
Connections:
- net labels added: +BATT, -BATT
- net labels removed: SOLAR_BACK_NEG, SOLAR_BACK_POS, SOLAR_FRONT_NEG, SOLAR_FRONT_POS, SOLAR_LEFT_NEG, SOLAR_LEFT_POS, SOLAR_RIGHT_NEG, SOLAR_RIGHT_POS
- wire segments 63 -> 101
Changed lines of the file:
@@
 Text Notes 6150 5000 0    60   ~ 0
 Exterior (rightmost) connector - pins 53 to 104
-Text Notes 3150 2100 0    60   ~ 0
+Text Notes 3150 2000 0    60   ~ 0
 Interior (leftmost) connector - pins 1 to 52
-Text Label 3850 3100 2    60   ~ 0
+Text Label 3000 3100 0    60   ~ 0
 He_UART_TX
 $Comp
@@
 U 1 1 5A568F72
 P 4050 3500
-F 0 "J?" H 4100 4917 50  0000 C CNN
-F 1 "Conn_02x26_Odd_Even" H 4100 4826 50  0000 C CNN
+F 0 "J?" H 4100 4950 50  0000 C CNN
+F 1 "Conn_02x26_Odd_Even" H 4100 4850 50  0000 C CNN
 F 2 "" H 4050 3500 50  0001 C CNN
 F 3 "~" H 4050 3500 50  0001 C CNN
@@
 	1    0    0    -1
 $EndComp
-Text Label 4350 3100 0    60   ~ 0
+Text Label 5200 3100 2    60   ~ 0
 He_UART_RX
 $Comp
@@
 Wire Wire Line
 	7550 3500 7500 3500
-Text Label 3850 2300 2    60   ~ 0
-SOLAR_FRONT_NEG
-Text Label 4350 2300 0    60   ~ 0
-SOLAR_FRONT_POS
-Text Label 3850 2400 2    60   ~ 0
-SOLAR_BACK_POS
-Text Label 3850 2500 2    60   ~ 0
-SOLAR_BACK_NEG
-Text Label 3850 2600 2    60   ~ 0
-SOLAR_LEFT_POS
-Text Label 3850 2700 2    60   ~ 0
-SOLAR_LEFT_NEG
-Text Label 3850 2800 2    60   ~ 0
-SOLAR_RIGHT_POS
-Text Label 3850 2900 2    60   ~ 0
-SOLAR_RIGHT_NEG
-Text Label 4350 2400 0    60   ~ 0
+Text Label 5200 2400 2    60   ~ 0
 1-WIRE
-Text Label 4350 2600 0    60   ~ 0
+Text Label 5200 2600 2    60   ~ 0
 BAT_HTR_EN_4
-Text Label 4350 2700 0    60   ~ 0
+Text Label 5200 2700 2    60   ~ 0
 BAT_HTR_EN_3
-Text Label 4350 2800 0    60   ~ 0
+Text Label 5200 2800 2    60   ~ 0
 BAT_HTR_EN_2
-Text Label 4350 2900 0    60   ~ 0
+Text Label 5200 2900 2    60   ~ 0
 BAT_HTR_EN_1
-Text Label 3850 3000 2    60   ~ 0
+Text Label 3000 3000 0    60   ~ 0
 ADC_INT
 $Comp
@@
 Wire Wire Line
 	4350 2450 4450 2450
-Text Label 4350 4200 0    60   ~ 0
+Text Label 5200 4200 2    60   ~ 0
 PAYLOAD_I_SENSE
 $Comp
@@
 Wire Wire Line
 	3850 4300 3800 4300
-Text Label 4350 4500 0    60   ~ 0
+Text Label 5200 4500 2    60   ~ 0
 He_EN
-Text Label 4350 4600 0    60   ~ 0
+Text Label 5200 4600 2    60   ~ 0
 PAYLOAD_EN
-Text Label 4350 4700 0    60   ~ 0
+Text Label 5200 4700 2    60   ~ 0
 PAYLOAD_HTR
-Text Label 4350 4800 0    60   ~ 0
+Text Label 5200 4800 2    60   ~ 0
 PAYLOAD_HTR
 $Comp
@@
 Wire Wire Line
 	4400 3850 4400 3900
-Text Label 4350 4100 0    60   ~ 0
+Text Label 5200 4100 2    60   ~ 0
 He_Tx_I_SENSE
 Wire Wire Line
@@
 Wire Wire Line
 	7550 4800 7500 4800
-Text Label 7500 4400 0    60   ~ 0
+Text Label 8350 4400 2    60   ~ 0
 PAYLOAD_ACT
-Text Label 7000 4400 2    60   ~ 0
+Text Label 6150 4400 0    60   ~ 0
 SC4
-Text Label 7000 4300 2    60   ~ 0
+Text Label 6150 4300 0    60   ~ 0
 SD4
 $Comp
@@
 Wire Wire Line
 	6950 2350 6950 2400
-Text Label 7000 2500 2    60   ~ 0
+Text Label 6150 2500 0    60   ~ 0
 SCL
-Text Label 7000 2600 2    60   ~ 0
+Text Label 6150 2600 0    60   ~ 0
 SDA
-Text Label 7000 2700 2    60   ~ 0
+Text Label 6150 2700 0    60   ~ 0
 BAT_HTR_MUX_SEL
-Text Label 7000 2800 2    60   ~ 0
+Text Label 6150 2800 0    60   ~ 0
 BAT_HTR_STAT_4
-Text Label 7000 2900 2    60   ~ 0
+Text Label 6150 2900 0    60   ~ 0
 BAT_HTR_STAT_3
-Text Label 7000 3000 2    60   ~ 0
+Text Label 6150 3000 0    60   ~ 0
 BAT_HTR_STAT_2
-Text Label 7000 3100 2    60   ~ 0
+Text Label 6150 3100 0    60   ~ 0
 BAT_HTR_STAT_1
-Text Label 7500 2600 0    60   ~ 0
+Text Label 8350 2600 2    60   ~ 0
 DEPLOYMENT_A
-Text Label 7500 2700 0    60   ~ 0
+Text Label 8350 2700 2    60   ~ 0
 DEPLOYMENT_B
-Text Label 7000 3200 2    60   ~ 0
+Text Label 6150 3200 0    60   ~ 0
 SDA_B
-Text Label 7000 3300 2    60   ~ 0
+Text Label 6150 3300 0    60   ~ 0
 SCL_B
+$Comp
+L power:+BATT #PWR?
+U 1 1 5A74D164
+P 3750 2300
+F 0 "#PWR?" H 3750 2150 50  0001 C CNN
+F 1 "+BATT" V 3765 2427 50  0000 L CNN
+F 2 "" H 3750 2300 50  0001 C CNN
+F 3 "" H 3750 2300 50  0001 C CNN
+	1    3750 2300
+	0    -1   -1   0
+$EndComp
+Wire Wire Line
+	3750 2300 3850 2300
+Wire Wire Line
+	3850 2300 3850 2200
+Wire Wire Line
+	3850 2200 4350 2200
+Wire Wire Line
+	4350 2200 4350 2300
+Connection ~ 3850 2300
+Wire Wire Line
+	3850 2300 3850 2400
+Wire Wire Line
+	3850 2400 3850 2500
+Connection ~ 3850 2400
+$Comp
+L power:-BATT #PWR?
+U 1 1 5A751FB0
+P 3750 2600
+F 0 "#PWR?" H 3750 2450 50  0001 C CNN
+F 1 "-BATT" V 3765 2727 50  0000 L CNN
+F 2 "" H 3750 2600 50  0001 C CNN
+F 3 "" H 3750 2600 50  0001 C CNN
+	1    3750 2600
+	0    -1   -1   0
+$EndComp
+Wire Wire Line
+	3750 2600 3850 2600
+Wire Wire Line
+	3850 2600 3850 2700
+Connection ~ 3850 2600
+Wire Wire Line
+	3850 2700 3850 2800
+Connection ~ 3850 2700
+Wire Wire Line
+	3850 2800 3850 2900
+Connection ~ 3850 2800
+Wire Wire Line
+	5200 4200 4350 4200
+Wire Wire Line
+	5200 4100 4350 4100
+Wire Wire Line
+	5200 2900 4350 2900
+Wire Wire Line
+	5200 2800 4350 2800
+Wire Wire Line
+	5200 2700 4350 2700
+Wire Wire Line
+	5200 2600 4350 2600
+Wire Wire Line
+	5200 2400 4350 2400
+Wire Wire Line
+	3850 3000 3000 3000
+Wire Wire Line
+	3850 3100 3000 3100
+Wire Wire Line
+	5200 4500 4350 4500
+Wire Wire Line
+	5200 4600 4350 4600
+Wire Wire Line
+	5200 4700 4350 4700
+Wire Wire Line
+	5200 4800 4350 4800
+Wire Wire Line
+	5200 3100 4350 3100
+Wire Wire Line
+	7000 2500 6150 2500
+Wire Wire Line
+	7000 2600 6150 2600
+Wire Wire Line
+	7000 2700 6150 2700
+Wire Wire Line
+	7000 2800 6150 2800
+Wire Wire Line
+	7000 2900 6150 2900
+Wire Wire Line
+	7000 3000 6150 3000
+Wire Wire Line
+	7000 3100 6150 3100
+Wire Wire Line
+	7000 3200 6150 3200
+Wire Wire Line
+	7000 3300 6150 3300
+Wire Wire Line
+	7000 4300 6150 4300
+Wire Wire Line
+	7000 4400 6150 4400
+Wire Wire Line
+	8350 4400 7500 4400
+Wire Wire Line
+	8350 2700 7500 2700
+Wire Wire Line
+	8350 2600 7500 2600
 $EndSCHEMATC

Commit message: Updated CubeSat board template
Connections:
- net labels added: MOTOR_CLK, MOTOR_CONF_CLK, MOTOR_CONF_DAT, MOTOR_CONF_LOAD, SDA_4, VPP
- net labels removed: -BATT, 1-WIRE, ADC_INT, He_Tx_I_SENSE, PAYLOAD_ACT, PAYLOAD_I_SENSE, SC4, SD4
Other:
- note added: "VAA = He_7V2"
- note added: "VPP = PAYLOAD_7V2"
Changed lines of the file:
@@
 Wire Wire Line
 	7550 3500 7500 3500
-Text Label 5200 2400 2    60   ~ 0
-1-WIRE
 Text Label 5200 2600 2    60   ~ 0
 BAT_HTR_EN_4
@@
 Text Label 5200 2900 2    60   ~ 0
 BAT_HTR_EN_1
-Text Label 3000 3000 0    60   ~ 0
-ADC_INT
 $Comp
 L power:+3V3 #PWR?
@@
 L power:GND #PWR?
 U 1 1 5A569CC3
-P 4450 2450
-F 0 "#PWR?" H 4450 2200 50  0001 C CNN
-F 1 "GND" V 4455 2322 50  0000 R CNN
-F 2 "" H 4450 2450 50  0001 C CNN
-F 3 "" H 4450 2450 50  0001 C CNN
-	1    4450 2450
+P 4450 2500
+F 0 "#PWR?" H 4450 2250 50  0001 C CNN
+F 1 "GND" V 4400 2600 50  0000 R CNN
+F 2 "" H 4450 2500 50  0001 C CNN
+F 3 "" H 4450 2500 50  0001 C CNN
+	1    4450 2500
 	0    -1   -1   0
 $EndComp
@@
 $EndComp
 Wire Wire Line
-	4350 2450 4350 2500
-Wire Wire Line
-	4350 2450 4450 2450
-Text Label 5200 4200 2    60   ~ 0
-PAYLOAD_I_SENSE
+	4350 2500 4450 2500
 $Comp
 L power:+3V3 #PWR?
@@
 Wire Wire Line
 	4400 3850 4400 3900
-Text Label 5200 4100 2    60   ~ 0
-He_Tx_I_SENSE
 Wire Wire Line
 	7500 4700 7550 4700
@@
 Wire Wire Line
 	7550 4800 7500 4800
-Text Label 8350 4400 2    60   ~ 0
-PAYLOAD_ACT
 Text Label 6150 4400 0    60   ~ 0
-SC4
+SDA_4
 Text Label 6150 4300 0    60   ~ 0
-SD4
+SDA_4
 $Comp
 L power:GND #PWR?
@@
 	3850 2400 3850 2500
 Connection ~ 3850 2400
-$Comp
-L power:-BATT #PWR?
-U 1 1 5A751FB0
+Wire Wire Line
+	5200 2900 4350 2900
+Wire Wire Line
+	5200 2800 4350 2800
+Wire Wire Line
+	5200 2700 4350 2700
+Wire Wire Line
+	5200 2600 4350 2600
+Wire Wire Line
+	3850 3100 3000 3100
+Wire Wire Line
+	5200 4500 4350 4500
+Wire Wire Line
+	5200 4600 4350 4600
+Wire Wire Line
+	5200 4700 4350 4700
+Wire Wire Line
+	5200 4800 4350 4800
+Wire Wire Line
+	5200 3100 4350 3100
+Wire Wire Line
+	7000 2500 6150 2500
+Wire Wire Line
+	7000 2600 6150 2600
+Wire Wire Line
+	7000 2700 6150 2700
+Wire Wire Line
+	7000 2800 6150 2800
+Wire Wire Line
+	7000 2900 6150 2900
+Wire Wire Line
+	7000 3000 6150 3000
+Wire Wire Line
+	7000 3100 6150 3100
+Wire Wire Line
+	7000 3200 6150 3200
+Wire Wire Line
+	7000 3300 6150 3300
+Wire Wire Line
+	7000 4300 6150 4300
+Wire Wire Line
+	7000 4400 6150 4400
+Wire Wire Line
+	8350 2700 7500 2700
+Wire Wire Line
+	8350 2600 7500 2600
+$Comp
+L power:GND #PWR?
+U 1 1 5A891B9F
 P 3750 2600
-F 0 "#PWR?" H 3750 2450 50  0001 C CNN
-F 1 "-BATT" V 3765 2727 50  0000 L CNN
+F 0 "#PWR?" H 3750 2350 50  0001 C CNN
+F 1 "GND" V 3755 2472 50  0000 R CNN
 F 2 "" H 3750 2600 50  0001 C CNN
 F 3 "" H 3750 2600 50  0001 C CNN
 	1    3750 2600
-	0    -1   -1   0
+	0    1    1    0
 $EndComp
 Wire Wire Line
@@
 	3850 2800 3850 2900
 Connection ~ 3850 2800
+Text Notes 7850 4550 0    60   ~ 0
+VAA = He_7V2
+$Comp
+L power:VPP #PWR?
+U 1 1 5A8A1847
+P 7550 4600
+F 0 "#PWR?" H 7550 4450 50  0001 C CNN
+F 1 "VPP" V 7565 4728 50  0000 L CNN
+F 2 "" H 7550 4600 50  0001 C CNN
+F 3 "" H 7550 4600 50  0001 C CNN
+	1    7550 4600
+	0    1    1    0
+$EndComp
+Wire Wire Line
+	7550 4600 7500 4600
+$Comp
+L power:VPP #PWR?
+U 1 1 5A8A4598
+P 6950 4600
+F 0 "#PWR?" H 6950 4450 50  0001 C CNN
+F 1 "VPP" V 6965 4727 50  0000 L CNN
+F 2 "" H 6950 4600 50  0001 C CNN
+F 3 "" H 6950 4600 50  0001 C CNN
+	1    6950 4600
+	0    -1   -1   0
+$EndComp
+Wire Wire Line
+	6950 4600 7000 4600
+Text Notes 7850 4650 0    60   ~ 0
+VPP = PAYLOAD_7V2
+Text Label 8350 4300 2    60   ~ 0
+MOTOR_CONF_LOAD
+Text Label 5200 4200 2    60   ~ 0
+MOTOR_CONF_CLK
+Text Label 5200 4100 2    60   ~ 0
+MOTOR_CONF_DAT
+Wire Wire Line
+	5200 4100 4350 4100
 Wire Wire Line
 	5200 4200 4350 4200
 Wire Wire Line
-	5200 4100 4350 4100
-Wire Wire Line
-	5200 2900 4350 2900
-Wire Wire Line
-	5200 2800 4350 2800
-Wire Wire Line
-	5200 2700 4350 2700
-Wire Wire Line
-	5200 2600 4350 2600
-Wire Wire Line
-	5200 2400 4350 2400
-Wire Wire Line
-	3850 3000 3000 3000
-Wire Wire Line
-	3850 3100 3000 3100
-Wire Wire Line
-	5200 4500 4350 4500
-Wire Wire Line
-	5200 4600 4350 4600
-Wire Wire Line
-	5200 4700 4350 4700
-Wire Wire Line
-	5200 4800 4350 4800
-Wire Wire Line
-	5200 3100 4350 3100
-Wire Wire Line
-	7000 2500 6150 2500
-Wire Wire Line
-	7000 2600 6150 2600
-Wire Wire Line
-	7000 2700 6150 2700
-Wire Wire Line
-	7000 2800 6150 2800
-Wire Wire Line
-	7000 2900 6150 2900
-Wire Wire Line
-	7000 3000 6150 3000
-Wire Wire Line
-	7000 3100 6150 3100
-Wire Wire Line
-	7000 3200 6150 3200
-Wire Wire Line
-	7000 3300 6150 3300
-Wire Wire Line
-	7000 4300 6150 4300
-Wire Wire Line
-	7000 4400 6150 4400
+	8350 4300 7500 4300
 Wire Wire Line
 	8350 4400 7500 4400
-Wire Wire Line
-	8350 2700 7500 2700
-Wire Wire Line
-	8350 2600 7500 2600
+Text Label 8350 4400 2    60   ~ 0
+MOTOR_CLK
 $EndSCHEMATC

Commit message: Replaced MOTOR_CONFIG channels with MOTOR_ENC channels
Connections:
- net labels added: MOTOR_ENC_A
- net labels removed: MOTOR_CONF_CLK, MOTOR_CONF_DAT
Changed lines of the file:
@@
 MOTOR_CONF_LOAD
 Text Label 5200 4200 2    60   ~ 0
-MOTOR_CONF_CLK
+MOTOR_ENC_A
 Text Label 5200 4100 2    60   ~ 0
-MOTOR_CONF_DAT
+MOTOR_ENC_A
 Wire Wire Line
 	5200 4100 4350 4100
